File: Hardware/RTC-Module.sch (EAGLE design)
At the start: 29 parts, among them J1 SMD, J2 SMD, J3 PTH, U2 RV-1805

Commit message: order protos, fix resistor PROD_ID
Parts:
- R6: value 1K -> 1k; device SparkFun-Resistors:2.55KOHM-0603-1/10W-1% -> SparkFun-Resistors:1KOHM-0603-1/10W-1%
Changed lines of the file:
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@@
 <part name="C3" library="SparkFun-Capacitors" deviceset="10NF" device="-0603-50V-10%" value="10nF"/>
 <part name="C4" library="SparkFun-Capacitors" deviceset="10NF" device="-0603-50V-10%" value="10nF"/>
-<part name="R6" library="SparkFun-Resistors" deviceset="2.55KOHM" device="-0603-1/10W-1%" value="1K"/>
+<part name="R6" library="SparkFun-Resistors" deviceset="1KOHM" device="-0603-1/10W-1%" value="1k"/>
 <part name="GND9" library="SparkFun" deviceset="GND" device=""/>
 <part name="SUPPLY1" library="SparkFun-PowerSymbols" deviceset="3.3V" device=""/>

Commit message: post checklist changes
Other:
- note added: "v10"
- note removed: "v02"
Changed lines of the file:
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@@
 <sheet>
 <plain>
-<text x="238.76" y="7.62" size="2.54" layer="94">v02</text>
+<text x="238.76" y="7.62" size="2.54" layer="94">v10</text>
 <text x="170.18" y="11.43" size="2.54" layer="94">A. England</text>
 <wire x1="0" y1="63.5" x2="106.68" y2="63.5" width="0.1524" layer="97" style="longdash"/>

Commit message: updated battery package
Parts:
- BT1: device SparkFun-Batteries:BATTERY-12MM_PTH -> Andy:BATTERY-12MM_PTH
Other:
- note added: "Optional Battery: PRT-07948"
Changed lines of the file:
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@@
 <part name="J4" library="SparkFun-Connectors" deviceset="CONN_03" device="1X03_NO_SILK"/>
 <part name="GND4" library="SparkFun" deviceset="GND" device=""/>
-<part name="BT1" library="SparkFun-Batteries" deviceset="BATTERY" device="-12MM_PTH"/>
+<part name="BT1" library="Andy" deviceset="BATTERY" device="-12MM_PTH"/>
 <part name="R5" library="SparkFun-Resistors" deviceset="470OHM" device="-0603-1/10W-1%" value="470"/>
 <part name="GND8" library="SparkFun" deviceset="GND" device=""/>
@@
 <sheet>
 <plain>
-<text x="238.76" y="7.62" size="2.54" layer="94">v10</text>
-<text x="170.18" y="11.43" size="2.54" layer="94">A. England</text>
+<text x="238.76" y="7.62" size="2.54" layer="94" font="vector">v10</text>
+<text x="170.18" y="11.43" size="2.54" layer="94" font="vector">A. England</text>
 <wire x1="0" y1="63.5" x2="106.68" y2="63.5" width="0.1524" layer="97" style="longdash"/>
 <wire x1="106.68" y1="63.5" x2="147.32" y2="63.5" width="0.1524" layer="97" style="longdash"/>
@@
 <text x="127" y="149.86" size="2.54" layer="97" font="vector">RTC Module</text>
 <text x="38.1" y="48.26" size="2.54" layer="97" font="vector">Qwiic Connectors/ I2C Interface</text>
-<text x="15.24" y="106.68" size="1.778" layer="97">Cut trace on jumper JP1
+<text x="15.24" y="106.68" size="1.778" layer="97" font="vector">Cut trace on jumper JP1
 to disconnect SuperCapacitor.
 Add solder to other side of
@@
 battery</text>
 <wire x1="147.32" y1="35.56" x2="147.32" y2="63.5" width="0.1524" layer="97" style="longdash"/>
-<text x="127" y="147.32" size="1.778" layer="97">Operating voltage: 1.5-3.6 V</text>
-<text x="193.04" y="142.24" size="1.778" layer="97">Disconnect I2C pullup
+<text x="127" y="147.32" size="1.778" layer="97" font="vector">Operating voltage: 1.5-3.6 V</text>
+<text x="193.04" y="142.24" size="1.778" layer="97" font="vector">Disconnect I2C pullup
 jumper if you already
 have pullup resistors
 on your I2C bus</text>
-<text x="127" y="144.78" size="1.778" layer="97">I2C Address: 0xD2</text>
+<text x="127" y="144.78" size="1.778" layer="97" font="vector">I2C Address: 0xD2</text>
+<text x="76.2" y="83.82" size="1.778" layer="97" font="vector">Optional Battery:
+PRT-07948</text>
 </plain>
 <instances>
@@
 <pinref part="J3" gate="G$1" pin="4"/>
 <wire x1="91.44" y1="35.56" x2="96.52" y2="35.56" width="0.1524" layer="91"/>
-<label x="96.52" y="35.56" size="1.27" layer="95" xref="yes"/>
-</segment>
-<segment>
-<label x="198.12" y="124.46" size="1.27" layer="95" xref="yes"/>
+<label x="96.52" y="35.56" size="1.27" layer="95" font="vector" xref="yes"/>
+</segment>
+<segment>
+<label x="198.12" y="124.46" size="1.27" layer="95" font="vector" xref="yes"/>
 <pinref part="R1" gate="G$1" pin="1"/>
 <wire x1="180.34" y1="124.46" x2="198.12" y2="124.46" width="0.1524" layer="91"/>
@@
 <pinref part="J3" gate="G$1" pin="3"/>
 <wire x1="91.44" y1="33.02" x2="96.52" y2="33.02" width="0.1524" layer="91"/>
-<label x="96.52" y="33.02" size="1.27" layer="95" xref="yes"/>
-</segment>
-<segment>
-<label x="198.12" y="121.92" size="1.27" layer="95" xref="yes"/>
+<label x="96.52" y="33.02" size="1.27" layer="95" font="vector" xref="yes"/>
+</segment>
+<segment>
+<label x="198.12" y="121.92" size="1.27" layer="95" font="vector" xref="yes"/>
 <pinref part="R2" gate="G$1" pin="1"/>
 <wire x1="195.58" y1="121.92" x2="198.12" y2="121.92" width="0.1524" layer="91"/>
@@
 <segment>
 <wire x1="177.8" y1="106.68" x2="208.28" y2="106.68" width="0.1524" layer="91"/>
-<label x="226.06" y="106.68" size="1.27" layer="95" xref="yes"/>
+<label x="226.06" y="106.68" size="1.27" layer="95" font="vector" xref="yes"/>
 <pinref part="R3" gate="G$1" pin="1"/>
 <wire x1="208.28" y1="106.68" x2="226.06" y2="106.68" width="0.1524" layer="91"/>
@@
 <segment>
 <wire x1="116.84" y1="35.56" x2="119.38" y2="35.56" width="0.1524" layer="91"/>
-<label x="119.38" y="35.56" size="1.27" layer="95" xref="yes"/>
+<label x="119.38" y="35.56" size="1.27" layer="95" font="vector" xref="yes"/>
 <pinref part="J4" gate="J$1" pin="3"/>
 </segment>
