File: Hardware/RTC-Module.brd (EAGLE design)
At the start: 25.4 x 25.4 mm, 27 parts, among them U2 RV-1805

Commit message: Changed pull ups, super cap silk, added panel.
Removed dupicate resistor on super cap. Removed pin 1 silk on super cap. Change I2C pull ups to 2.2k for 3.3V devices. Changed pull ups to 10k for lower draw. Added panel.
Parts:
- removed R5: 2.55k, SparkFun-Resistors:0603
- C1: device SparkFun-Capacitors:DSK-RADIAL-4.8MM -> SparkFun-Capacitors:DSK-RADIAL-6.8MM
- J1, J2: value (none) -> SMD
- J3: value (none) -> PTH
- R1, R2: value 4.7k -> 2.2k; device SparkFun-Resistors:0603@1 -> SparkFun-Resistors:0603
- R3, R4, R7: value 4.7k -> 10k; device SparkFun-Resistors:0603@1 -> SparkFun-Resistors:0603
- R6: value 2.55k -> 1K
- U$3: value SPARKX-LOGO2 -> SPARKX-LOGO4; device SparkX:SPARKX-TINY -> SparkX:SPARKX-MEDIUM
- moved U$3 17.6 mm to (12.7, 22.1)
Connections:
- net N$5: no longer R5.1
- net VBACKUP: no longer R5.2
Routing:
- net VBACKUP: track 20.6 -> 16.8 mm
- net N$5: track 7.19 -> 4.65 mm

Commit message: laying out with battery
Parts:
- removed U$3, U$5: SPARKX-LOGO4, SparkX:SPARKX-MEDIUM
- added BT1: (no value), SparkFun-Batteries:BATTCON_12MM_PTH
- added JP1: JUMPER-SMT_3_1-NC_TRACE_NO-SILK, SparkFun-Jumpers:SMT-JUMPER_3_1-NC_TRACE_NO-SILK
- added R5: 470, SparkFun-Resistors:0603
- moved R7 20.4 mm to (22.9, 17.1), turned to 0 degrees
- moved R6 17.8 mm to (2.54, 17.1), turned to 0 degrees
- moved R4 17.8 mm to (22.9, 19.1), turned to 0 degrees
- moved R1 8.26 mm to (8.26, 6.35)
- moved R2 8.25 mm to (17.1, 6.35)
- moved FD1 7.14 mm to (19.7, 24.6)
- moved FD2 7.14 mm to (19.7, 24.6)
- moved C1 2.16 mm to (12.7, 15.0)
- moved U2 1.90 mm to (12.7, 9.53)
- moved C2 0.65 mm to (8.26, 8.89)
- moved R3 0.65 mm to (17.1, 8.89)
- moved C4 0.63 mm to (8.26, 11.4), turned to 180 degrees
- moved SJ2 0.63 mm to (12.7, 5.71), turned to 180 degrees
- moved C3 0.63 mm to (17.1, 11.4), turned to 0 degrees
Connections:
- new net N$3: BT1.VCC@1, R5.1
- new net N$6: C1.+, JP1.3
- new net N$7: JP1.1, R5.2
- net GND: now also BT1.GND
- net N$5: now also JP1.2; no longer C1.+
Routing:
- net 3.3V: track 65.1 -> 27.2 mm, vias 5 -> 2
- net !RST: track 34.9 -> 19.5 mm, vias 1 -> 0
- net N$6: track 0.00 -> 15.2 mm, vias 0 -> 1
- net PSW: track 41.1 -> 27.4 mm, vias 1 -> 3
- net SDA: track 36.5 -> 25.6 mm, vias 0 -> 3
- net N$7: track 0.00 -> 7.39 mm, vias 0 -> 1
- net SCL: track 37.2 -> 30.8 mm, vias 3 -> 2
- net N$2: track 2.15 -> 5.25 mm
- net N$1: track 2.15 -> 5.25 mm
- net N$3: track 0.00 -> 2.76 mm
- net VBACKUP: track 16.8 -> 19.1 mm, vias 0 -> 2
- net N$4: track 5.73 -> 3.67 mm
- net !INT: track 14.6 -> 16.1 mm
- net N$5: track 4.65 -> 5.94 mm, vias 0 -> 1

Commit message: added battery footprint, went through engineering checklist
Parts:
- added LOGO2, LOGO3: SFE_LOGO_NAME_FLAME.1_INCH, SparkFun-Aesthetics:SFE_LOGO_NAME_FLAME_.1
Routing:
- net 3.3V: track 27.2 -> 80.5 mm, vias 2 -> 3
- net !RST: track 19.5 -> 41.6 mm, vias 0 -> 1
- net SDA: track 25.6 -> 43.5 mm, vias 3 -> 4
- net SCL: track 30.8 -> 39.2 mm
- net VBACKUP: track 19.1 -> 20.3 mm
- net N$5: track 5.94 -> 6.45 mm
Other:
- board text added: "B"
- board text added: "C"
- board text added: "v02"
- board text removed: "X01"

Commit message: post review changes
Parts:
- moved LOGO3 7.62 mm to (18.7, 6.73)
Changed lines of the file:
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@@
 <layer number="20" name="Dimension" color="15" fill="1" visible="yes" active="yes"/>
 <layer number="21" name="tPlace" color="16" fill="1" visible="yes" active="yes"/>
-<layer number="22" name="bPlace" color="14" fill="1" visible="yes" active="yes"/>
+<layer number="22" name="bPlace" color="14" fill="1" visible="no" active="yes"/>
 <layer number="23" name="tOrigins" color="15" fill="1" visible="yes" active="yes"/>
-<layer number="24" name="bOrigins" color="15" fill="1" visible="yes" active="yes"/>
+<layer number="24" name="bOrigins" color="15" fill="1" visible="no" active="yes"/>
 <layer number="25" name="tNames" color="7" fill="1" visible="yes" active="yes"/>
 <layer number="26" name="bNames" color="7" fill="1" visible="no" active="yes"/>
@@
 <layer number="29" name="tStop" color="7" fill="3" visible="no" active="yes"/>
 <layer number="30" name="bStop" color="7" fill="6" visible="no" active="yes"/>
-<layer number="31" name="tCream" color="7" fill="4" visible="yes" active="yes"/>
-<layer number="32" name="bCream" color="7" fill="5" visible="yes" active="yes"/>
+<layer number="31" name="tCream" color="7" fill="4" visible="no" active="yes"/>
+<layer number="32" name="bCream" color="7" fill="5" visible="no" active="yes"/>
 <layer number="33" name="tFinish" color="6" fill="3" visible="no" active="yes"/>
 <layer number="34" name="bFinish" color="6" fill="6" visible="no" active="yes"/>
@@
 <layer number="37" name="tTest" color="7" fill="1" visible="no" active="yes"/>
 <layer number="38" name="bTest" color="7" fill="1" visible="no" active="yes"/>
-<layer number="39" name="tKeepout" color="4" fill="11" visible="yes" active="yes"/>
-<layer number="40" name="bKeepout" color="1" fill="11" visible="yes" active="yes"/>
+<layer number="39" name="tKeepout" color="4" fill="11" visible="no" active="yes"/>
+<layer number="40" name="bKeepout" color="1" fill="11" visible="no" active="yes"/>
 <layer number="41" name="tRestrict" color="4" fill="10" visible="no" active="yes"/>
 <layer number="42" name="bRestrict" color="1" fill="10" visible="no" active="yes"/>
@@
 <layer number="45" name="Holes" color="7" fill="1" visible="no" active="yes"/>
 <layer number="46" name="Milling" color="3" fill="1" visible="no" active="yes"/>
-<layer number="47" name="Measures" color="7" fill="1" visible="yes" active="yes"/>
+<layer number="47" name="Measures" color="7" fill="1" visible="no" active="yes"/>
 <layer number="48" name="Document" color="7" fill="1" visible="no" active="yes"/>
 <layer number="49" name="Reference" color="7" fill="1" visible="no" active="yes"/>
 <layer number="50" name="dxf" color="7" fill="1" visible="no" active="no"/>
-<layer number="51" name="tDocu" color="6" fill="1" visible="yes" active="yes"/>
+<layer number="51" name="tDocu" color="6" fill="1" visible="no" active="yes"/>
 <layer number="52" name="bDocu" color="7" fill="1" visible="no" active="yes"/>
 <layer number="53" name="tGND_GNDA" color="7" fill="9" visible="no" active="no"/>
@@
 RTC
 Module</text>
-<text x="12.573" y="8.89" size="1.27" layer="22" font="vector" ratio="15" rot="MR0" align="center">Qwiic RTC Module</text>
+<text x="12.573" y="6.35" size="1.27" layer="22" font="vector" ratio="15" rot="MR0" align="center">Qwiic RTC Module</text>
 <text x="10.16" y="2.413" size="0.8128" layer="21" font="vector" ratio="15" rot="R90" align="center-left">SDA</text>
 <text x="12.7" y="2.413" size="0.8128" layer="21" font="vector" ratio="15" rot="R90" align="center-left">SCL</text>
@@
 <element name="JP1" library="SparkFun-Jumpers" package="SMT-JUMPER_3_1-NC_TRACE_NO-SILK" value="JUMPER-SMT_3_1-NC_TRACE_NO-SILK" x="2.54" y="15.24" rot="MR180"/>
 <element name="LOGO2" library="SparkFun-Aesthetics" package="SFE_LOGO_NAME_FLAME_.1" value="SFE_LOGO_NAME_FLAME.1_INCH" x="6.858" y="19.812"/>
-<element name="LOGO3" library="SparkFun-Aesthetics" package="SFE_LOGO_NAME_FLAME_.1" value="SFE_LOGO_NAME_FLAME.1_INCH" x="18.669" y="14.351" rot="MR0"/>
+<element name="LOGO3" library="SparkFun-Aesthetics" package="SFE_LOGO_NAME_FLAME_.1" value="SFE_LOGO_NAME_FLAME.1_INCH" x="18.669" y="6.731" rot="MR0"/>
 </elements>
 <signals>
