File: Hardware/RTC-Module.brd (EAGLE design)
At the start: 25.4 x 25.4 mm, 29 parts, among them J1 SMD, J2 SMD, J3 PTH, U2 RV-1805

Commit message: order protos, fix resistor PROD_ID
Parts:
- R6: value 1K -> 1k
Changed lines of the file:
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@@
 <attribute name="PROD_ID" value="CAP-00867" x="8.255" y="11.43" size="1.778" layer="27" rot="R180" display="off"/>
 </element>
-<element name="R6" library="SparkFun-Resistors" package="0603" value="1K" x="2.54" y="17.145">
-<attribute name="PROD_ID" value="RES-11227" x="2.54" y="17.145" size="1.778" layer="27" display="off"/>
+<element name="R6" library="SparkFun-Resistors" package="0603" value="1k" x="2.54" y="17.145">
+<attribute name="PROD_ID" value="RES-07856" x="2.54" y="17.145" size="1.778" layer="27" display="off"/>
 </element>
 <element name="R4" library="SparkFun-Resistors" package="0603" value="10k" x="22.86" y="19.05">

Commit message: post checklist changes
Routing:
- net N$5: track 6.45 -> 5.54 mm
Other:
- board text added: "BAT"
- board text added: "CAP"
- board text added: "PWR"
- board text added: "Units in Inches"
- board text added: "v10"
- board text removed: "B"
- board text removed: "C"
- board text removed: "v02"
Changed lines of the file:
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@@
 <layer number="20" name="Dimension" color="15" fill="1" visible="yes" active="yes"/>
 <layer number="21" name="tPlace" color="16" fill="1" visible="yes" active="yes"/>
-<layer number="22" name="bPlace" color="14" fill="1" visible="yes" active="yes"/>
+<layer number="22" name="bPlace" color="14" fill="1" visible="no" active="yes"/>
 <layer number="23" name="tOrigins" color="15" fill="1" visible="yes" active="yes"/>
 <layer number="24" name="bOrigins" color="15" fill="1" visible="no" active="yes"/>
@@
 <layer number="37" name="tTest" color="7" fill="1" visible="no" active="yes"/>
 <layer number="38" name="bTest" color="7" fill="1" visible="no" active="yes"/>
-<layer number="39" name="tKeepout" color="4" fill="11" visible="no" active="yes"/>
-<layer number="40" name="bKeepout" color="1" fill="11" visible="no" active="yes"/>
+<layer number="39" name="tKeepout" color="4" fill="11" visible="yes" active="yes"/>
+<layer number="40" name="bKeepout" color="1" fill="11" visible="yes" active="yes"/>
 <layer number="41" name="tRestrict" color="4" fill="10" visible="no" active="yes"/>
 <layer number="42" name="bRestrict" color="1" fill="10" visible="no" active="yes"/>
@@
 <layer number="45" name="Holes" color="7" fill="1" visible="no" active="yes"/>
 <layer number="46" name="Milling" color="3" fill="1" visible="no" active="yes"/>
-<layer number="47" name="Measures" color="7" fill="1" visible="no" active="yes"/>
+<layer number="47" name="Measures" color="7" fill="1" visible="yes" active="yes"/>
 <layer number="48" name="Document" color="7" fill="1" visible="no" active="yes"/>
 <layer number="49" name="Reference" color="7" fill="1" visible="no" active="yes"/>
 <layer number="50" name="dxf" color="7" fill="1" visible="no" active="no"/>
-<layer number="51" name="tDocu" color="6" fill="1" visible="no" active="yes"/>
+<layer number="51" name="tDocu" color="6" fill="1" visible="yes" active="yes"/>
 <layer number="52" name="bDocu" color="7" fill="1" visible="no" active="yes"/>
 <layer number="53" name="tGND_GNDA" color="7" fill="9" visible="no" active="no"/>
@@
 <wire x1="25.4" y1="0" x2="25.4" y2="25.4" width="0.2032" layer="20"/>
 <text x="12.7" y="7.366" size="0.8128" layer="21" font="vector" ratio="15" rot="R180" align="center">I2C</text>
-<text x="24.892" y="0.508" size="1.27" layer="16" font="vector" ratio="15" rot="MR0">v02</text>
+<text x="24.892" y="0.508" size="1.27" layer="16" font="vector" ratio="15" rot="MR0">v10</text>
 <text x="17.78" y="-8.89" size="1.778" layer="51">Andy England</text>
 <dimension x1="0" y1="25.4" x2="0" y2="0" x3="-7.62" y3="12.7" textsize="1.016" textratio="15" layer="47" unit="inch"/>
@@
 <text x="17.78" y="2.413" size="0.8128" layer="22" font="vector" ratio="15" rot="MR90" align="center-left">!INT</text>
 <text x="20.32" y="2.413" size="0.8128" layer="22" font="vector" ratio="15" rot="MR90" align="center-left">!RST</text>
-<text x="1.778" y="16.383" size="0.8128" layer="22" font="vector" ratio="15" rot="MR0">B</text>
-<text x="3.81" y="16.256" size="0.8128" layer="22" font="vector" ratio="15" rot="MR0">C</text>
+<text x="1.905" y="14.478" size="0.8128" layer="22" font="vector" ratio="15" rot="MR270">BAT</text>
+<text x="3.937" y="14.478" size="0.8128" layer="22" font="vector" ratio="15" rot="MR270">CAP</text>
+<text x="3.556" y="16.256" size="0.8128" layer="22" font="vector" ratio="15" rot="MR0">PWR</text>
+<text x="12.7" y="34.29" size="1.016" layer="47" font="vector" align="center">Units in Inches</text>
 </plain>
 <attributes>
@@
 <via x="7.239" y="10.16" extent="1-16" drill="0.381"/>
 <via x="5.588" y="16.383" extent="1-16" drill="0.381"/>
-<via x="3.683" y="13.843" extent="1-16" drill="0.381"/>
+<via x="1.905" y="11.811" extent="1-16" drill="0.381"/>
 <via x="9.779" y="10.16" extent="1-16" drill="0.381"/>
 <via x="14.986" y="11.557" extent="1-16" drill="0.381"/>
@@
 <wire x1="1.69" y1="17.145" x2="2.413" y2="17.145" width="0.2032" layer="1"/>
 <wire x1="2.413" y1="17.145" x2="2.54" y2="17.018" width="0.2032" layer="1"/>
+<via x="2.54" y="13.97" extent="1-16" drill="0.381"/>
+<wire x1="2.54" y1="13.97" x2="2.54" y2="15.24" width="0.2032" layer="16"/>
 <wire x1="2.54" y1="17.018" x2="2.54" y2="16.51" width="0.2032" layer="1"/>
-<wire x1="2.54" y1="16.51" x2="2.794" y2="16.256" width="0.2032" layer="1"/>
-<via x="2.54" y="13.462" extent="1-16" drill="0.381"/>
-<wire x1="2.54" y1="13.462" x2="2.54" y2="15.24" width="0.2032" layer="16"/>
-<wire x1="2.794" y1="16.256" x2="2.794" y2="13.716" width="0.2032" layer="1"/>
-<wire x1="2.794" y1="13.716" x2="2.54" y2="13.462" width="0.2032" layer="1"/>
+<wire x1="2.54" y1="16.51" x2="2.921" y2="16.129" width="0.2032" layer="1"/>
+<wire x1="2.921" y1="16.129" x2="2.921" y2="14.351" width="0.2032" layer="1"/>
+<wire x1="2.921" y1="14.351" x2="2.54" y2="13.97" width="0.2032" layer="1"/>
 </signal>
 <signal name="N$6">

Commit message: updated battery package
Parts:
- BT1: device SparkFun-Batteries:BATTCON_12MM_PTH -> Andy:BATTCON_12MM_PTH
Changed lines of the file:
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@@
 <layer number="27" name="tValues" color="7" fill="1" visible="no" active="yes"/>
 <layer number="28" name="bValues" color="7" fill="1" visible="no" active="yes"/>
-<layer number="29" name="tStop" color="7" fill="3" visible="no" active="yes"/>
-<layer number="30" name="bStop" color="7" fill="6" visible="no" active="yes"/>
+<layer number="29" name="tStop" color="7" fill="3" visible="yes" active="yes"/>
+<layer number="30" name="bStop" color="7" fill="6" visible="yes" active="yes"/>
 <layer number="31" name="tCream" color="7" fill="4" visible="no" active="yes"/>
 <layer number="32" name="bCream" color="7" fill="5" visible="no" active="yes"/>
@@
 <text x="12.7" y="7.366" size="0.8128" layer="21" font="vector" ratio="15" rot="R180" align="center">I2C</text>
 <text x="24.892" y="0.508" size="1.27" layer="16" font="vector" ratio="15" rot="MR0">v10</text>
-<text x="17.78" y="-8.89" size="1.778" layer="51">Andy England</text>
+<text x="17.78" y="-8.89" size="1.778" layer="51" font="vector">Andy England</text>
 <dimension x1="0" y1="25.4" x2="0" y2="0" x3="-7.62" y3="12.7" textsize="1.016" textratio="15" layer="47" unit="inch"/>
 <dimension x1="2.54" y1="22.86" x2="2.54" y2="0" x3="-3.81" y3="11.43" textsize="1.016" textratio="15" layer="47" unit="inch"/>
@@
 </element>
 <element name="J4" library="SparkFun-Connectors" package="1X03_NO_SILK" value="" x="20.32" y="1.27" rot="R180"/>
-<element name="BT1" library="SparkFun-Batteries" package="BATTCON_12MM_PTH" value="" x="12.7" y="19.177" rot="MR0">
+<element name="BT1" library="Andy" package="BATTCON_12MM_PTH" value="" x="12.7" y="19.177" rot="MR0">
 <attribute name="SF_SKU" value="PRT-07948" x="12.7" y="19.177" size="1.778" layer="28" rot="MR0" display="off"/>
 <attribute name="PROD_ID" value="BATT-08315" x="12.7" y="19.177" size="1.778" layer="28" rot="MR0" display="off"/>
